Commit message: minor fixes removing shakiness in gazebo

File: src/manipulator_description/urdf/ur5_robotiq_joint_limited_robot.urdf.xacro (robot description, xacro)
@@ -12,5 +12,5 @@
     <parent link="world" />
     <child link = "base_link" />
-    <origin xyz="0.0 0.0 0.0" rpy="0.0 0.0 0.0" />
+    <origin xyz="0.0 0.0 0.0" rpy="0.0 0.0 -1.570" />
   </joint>
   <!-- arm top table-->
@@ -18,5 +18,5 @@
     <parent link="world"/>
     <child link="table_top_link" />
-    <origin xyz="-${table_x} +0.21 -${table_height}" rpy="0.0 0.0 0.0" />
+    <origin xyz="-${table_x} +0.21 -${table_height+0.005}" rpy="0.0 0.0 0.0" />
   </joint>
   <xacro:ur5_robot prefix="" joint_limited="true"/>
